Commit message: PR2 updates

File: models/drake/iiwa_description/urdf/iiwa14_polytope_collision.urdf (robot description, URDF)
Before this commit: robot iiwa14, 11 links, 10 joints
Links:
- link iiwa_link_6: geometry collision mesh filename=../meshes/collision/link_6.obj; visual mesh filename=../meshes/visual/link_6.obj
